Commit message: LeArm: Update MoveIt configuration
- Regenerate off latest URDF.
- Edit joint_limts.yaml to enable acceleration limits - required by rviz tool.

Signed-off-by: Rhys Mainwaring <rhys.mainwaring@me.com>

File: learm_moveit_config/config/learm.ros2_control.xacro (robot description, xacro)
@@ -50,39 +50,4 @@
                 <state_interface name="velocity"/>
             </joint>
-            <joint name="finger_left">
-                <command_interface name="position"/>
-                <state_interface name="position">
-                  <param name="initial_value">${initial_positions['finger_left']}</param>
-                </state_interface>
-                <state_interface name="velocity"/>
-            </joint>
-            <joint name="grip_right">
-                <command_interface name="position"/>
-                <state_interface name="position">
-                  <param name="initial_value">${initial_positions['grip_right']}</param>
-                </state_interface>
-                <state_interface name="velocity"/>
-            </joint>
-            <joint name="finger_right">
-                <command_interface name="position"/>
-                <state_interface name="position">
-                  <param name="initial_value">${initial_positions['finger_right']}</param>
-                </state_interface>
-                <state_interface name="velocity"/>
-            </joint>
-            <joint name="tendon_left">
-                <command_interface name="position"/>
-                <state_interface name="position">
-                  <param name="initial_value">${initial_positions['tendon_left']}</param>
-                </state_interface>
-                <state_interface name="velocity"/>
-            </joint>
-            <joint name="tendon_right">
-                <command_interface name="position"/>
-                <state_interface name="position">
-                  <param name="initial_value">${initial_positions['tendon_right']}</param>
-                </state_interface>
-                <state_interface name="velocity"/>
-            </joint>
         </ros2_control>
     </xacro:macro>
