Commit message: LeArm: Update URDF generated from SDF
Signed-off-by: Rhys Mainwaring <rhys.mainwaring@me.com>

File: ardupilot_gz_description/models/learm/model.urdf (robot description, URDF)
Before this commit: robot learm, 14 links, 13 joints
Links:
- removed link camera_link
- removed link camera_wrist_link
- link finger_left_link: geometry collision box size=0.005 0.01 0.06; visual mesh filename=package://ardupilot_gz_description/models/learm/meshes/fing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 scale=1 1 1
- link finger_right_link: geometry collision box size=0.005 0.01 0.06; visual mesh filename=package://ardupilot_gz_description/models/learm/meshes/fing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 scale=1 1 1
- link forearm_link: mass 0.0396626 -> 0.03636; geometry collision box size=0.025 0.04 0.06; visual mesh filename=package://ardupilot_gz_description/models/learm/meshes/fore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 scale=1 1 1
- link grip_left_link: geometry collision box size=0.004 0.015 0.04; visual mesh filename=package://ardupilot_gz_description/models/learm/meshes/carp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 scale=1 1 1
- link grip_right_link: geometry collision box size=0.005 0.015 0.04; visual mesh filename=package://ardupilot_gz_description/models/learm/meshes/carp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 scale=1 1 1
- link hand_link: mass 0.06464 -> 0.03232; geometry collision box size=0.04 0.04 0.02; visual mesh filename=package://ardupilot_gz_description/models/learm/meshes/hand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 scale=1 1 1
- link humerus_link: geometry collision box size=0.025 0.05 0.08; visual mesh filename=package://ardupilot_gz_description/models/learm/meshes/hume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 scale=1 1 1
- link shoulder_link: mass 0.02424 -> 0.0253841; geometry collision cylinder length=0.025 radius=0.04; visual mesh filename=package://ardupilot_gz_description/models/learm/meshes/shou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 scale=1 1 1
- link wrist_link: geometry collision box size=0.04 0.03 0.06; visual mesh filename=package://ardupilot_gz_description/models/learm/meshes/wris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 scale=1 1 1
Joints:
- removed joint camera_base_joint
- removed joint camera_wrist_joint
- joint elbow: limit lower=-1.57 upper=1.57 effort=inf velocity=inf -> lower=-1.57 upper=1.57 effort=10 velocity=0.5
- joint finger_left: limit lower=0 upper=1.57 effort=inf velocity=inf -> lower=0 upper=1.57 effort=10 velocity=0.5
- joint finger_right: limit lower=0 upper=1.57 effort=inf velocity=inf -> lower=0 upper=1.57 effort=10 velocity=0.5
- joint grip_left: limit lower=0 upper=1.57 effort=inf velocity=inf -> lower=0 upper=1.57 effort=10 velocity=0.5
- joint grip_right: limit lower=0 upper=1.57 effort=inf velocity=inf -> lower=0 upper=1.57 effort=10 velocity=0.5
- joint shoulder_lift: limit lower=-3.142 upper=0 effort=inf velocity=inf -> lower=-3.142 upper=0 effort=50 velocity=0.5
- joint shoulder_pan: limit lower=-1.57 upper=1.57 effort=inf velocity=inf -> lower=-1.57 upper=1.57 effort=10 velocity=0.5
- joint tendon_left: limit lower=0 upper=1.57 effort=inf velocity=inf -> lower=0 upper=1.57 effort=10 velocity=0.5
- joint tendon_right: limit lower=0 upper=1.57 effort=inf velocity=inf -> lower=0 upper=1.57 effort=10 velocity=0.5
- joint wrist_flex: limit lower=-1.57 upper=1.57 effort=inf velocity=inf -> lower=-1.57 upper=1.57 effort=10 velocity=0.5
- joint wrist_roll: limit lower=-1.57 upper=1.57 effort=inf velocity=inf -> lower=-1.57 upper=1.57 effort=10 velocity=0.5

Commit message: LeArm: Use collada visual and low poly collision meshes in urdf
Signed-off-by: Rhys Mainwaring <rhys.mainwaring@me.com>

File: ardupilot_gz_description/models/learm/model.urdf (robot description, URDF)
Before this commit: robot learm, 12 links, 11 joints
Links:
- link arm_base_link: geometry collision cylinder length=0.08 radius=0.06; visual mesh filename=package://ardupilot_gz_description/models/learm/meshes/base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 scale=1 1 1
- link finger_left_link: geometry collision mesh filename=package://ardupilot_gz_description/models/learm/meshes/fing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 scale=1 1 1; visual mesh filename=package://ardupilot_gz_description/models/learm/meshes/fing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 scale=1 1 1
- link finger_right_link: geometry collision mesh filename=package://ardupilot_gz_description/models/learm/meshes/fing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 scale=1 1 1; visual mesh filename=package://ardupilot_gz_description/models/learm/meshes/fing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 scale=1 1 1
- link forearm_link: geometry collision mesh filename=package://ardupilot_gz_description/models/learm/meshes/fore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 scale=1 1 1; visual mesh filename=package://ardupilot_gz_description/models/learm/meshes/fore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 scale=1 1 1
- link grip_left_link: geometry collision mesh filename=package://ardupilot_gz_description/models/learm/meshes/carp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 scale=1 1 1; visual mesh filename=package://ardupilot_gz_description/models/learm/meshes/carp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 scale=1 1 1
- link grip_right_link: geometry collision mesh filename=package://ardupilot_gz_description/models/learm/meshes/carp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 scale=1 1 1; visual mesh filename=package://ardupilot_gz_description/models/learm/meshes/carp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 scale=1 1 1
- link hand_link: geometry collision mesh filename=package://ardupilot_gz_description/models/learm/meshes/hand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 scale=1 1 1; visual mesh filename=package://ardupilot_gz_description/models/learm/meshes/hand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 scale=1 1 1
- link humerus_link: geometry collision mesh filename=package://ardupilot_gz_description/models/learm/meshes/hume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 scale=1 1 1; visual mesh filename=package://ardupilot_gz_description/models/learm/meshes/hume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 scale=1 1 1
- link shoulder_link: geometry collision mesh filename=package://ardupilot_gz_description/models/learm/meshes/shou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 scale=1 1 1; visual mesh filename=package://ardupilot_gz_description/models/learm/meshes/shou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 scale=1 1 1
- link wrist_link: geometry collision mesh filename=package://ardupilot_gz_description/models/learm/meshes/wris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 scale=1 1 1; visual mesh filename=package://ardupilot_gz_description/models/learm/meshes/wris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 scale=1 1 1
