Commit message: iris_with_arm: update generated urdf model
- Rerun script and save updated copy of the generated urdf.

Signed-off-by: Rhys Mainwaring <rhys.mainwaring@me.com>

File: ardupilot_gz_description/models/iris_with_arm/model.urdf (robot description, URDF)
Before this commit: robot iris_with_arm, 13 links, 12 joints
Links:
- link arm_Fixed_Gripper: geometry collision mesh filename=package://so_arm_100_description/models/so_arm_100_5dof/mes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 scale=0.9 0.9 0.9; visual box size=0.01 0.01 0.01
- link arm_Lower_Arm: geometry collision mesh filename=package://so_arm_100_description/models/so_arm_100_5dof/mes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 scale=0.9 0.9 0.9; visual mesh filename=package://so_arm_100_description/models/so_arm_100_5dof/mes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 scale=1 1 1
- link arm_Moving_Jaw: geometry collision mesh filename=package://so_arm_100_description/models/so_arm_100_5dof/mes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 scale=0.9 0.9 0.9; visual mesh filename=package://so_arm_100_description/models/so_arm_100_5dof/mes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 scale=1 1 1
- link arm_Shoulder_Rotation_Pitch: geometry collision mesh filename=package://so_arm_100_description/models/so_arm_100_5dof/mes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 scale=0.9 0.9 0.9; visual mesh filename=package://so_arm_100_description/models/so_arm_100_5dof/mes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 scale=1 1 1
- link arm_Upper_Arm: geometry collision mesh filename=package://so_arm_100_description/models/so_arm_100_5dof/mes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 scale=0.9 0.9 0.9; visual mesh filename=package://so_arm_100_description/models/so_arm_100_5dof/mes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 scale=1 1 1
- link arm_Wrist_Pitch_Roll: geometry collision mesh filename=package://so_arm_100_description/models/so_arm_100_5dof/mes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 scale=0.9 0.9 0.9; visual mesh filename=package://so_arm_100_description/models/so_arm_100_5dof/mes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 scale=1 1 1
- link arm_base_link: geometry collision mesh filename=package://so_arm_100_description/models/so_arm_100_5dof/mes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 scale=0.9 0.9 0.9; visual mesh filename=package://so_arm_100_description/models/so_arm_100_5dof/mes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 scale=1 1 1

Commit message: iris_with_arm: update generated urdf model
- Use updated collisions

Signed-off-by: Rhys Mainwaring <rhys.mainwaring@me.com>

File: ardupilot_gz_description/models/iris_with_arm/model.urdf (robot description, URDF)
Before this commit: robot iris_with_arm, 13 links, 12 joints
Links:
- link base_link: geometry collision cylinder length=0.17 radius=0.005; collision cylinder length=0.17 radius=0.005
